File: sensor-gnss-neo6mv2/sensor-gnss-neo6mv2.kicad_pcb (KiCad board)
At the start: 2 copper layers, 38.7 x 45 mm, 7 parts, among them J1 PWR, J2 ESP-01S, J3 NEO6M, U1 LMZM23601V3SILR

Commit message: First prototype sent to production
Parts:
- moved D1 29.3 mm to (130.6, 99.5), turned to 0 degrees
- moved Cin1 25.8 mm to (130.7, 96.4), turned to 0 degrees
- moved U1 20.4 mm to (130.6, 90.9), turned to 90 degrees
- moved Cout1 17.4 mm to (130.5, 86.0), turned to 0 degrees
- moved J3 0.24 mm to (116.3, 71.7)
Connections:
- net Net-(D1-A) renamed /PWR VCC
- net Net-(J2-RX) renamed /Data
- J2 pad 2: Net-(J2-TX) -> unconnected-(J2-TX-Pad2)
- J3 pad 2: Net-(J2-TX) -> unconnected-(J3-RX-Pad2)
Routing:
- net /PWR VCC: track 34.1 -> 12.9 mm
- net Net-(J2-TX): track 19.0 -> 0.00 mm
- net +3V3: track 68.0 -> 58.6 mm

Commit message: v3, revised based on first proto version
Parts:
- J1: footprint TerminalBlock_MetzConnect:TerminalBlock_MetzConnect_Type086_RT03402HBLC_1x02_P3.81mm_Horizontal -> C5349550:CONN-TH_MX127S-3.81-02P-GN01-CU-Y-A
- moved J1 1.94 mm to (144.0, 95.9)
Routing:
- net +3V3: track 58.6 -> 73.3 mm
- net /PWR VCC: track 12.9 -> 24.5 mm
- net Earth: track 23.8 -> 30.3 mm
- net /Data: track 34.7 -> 35.6 mm
Other:
- board size 38.7 x 45 mm -> 40 x 45 mm
- board text added: "3V3"
- board text added: "GND"
- board text added: "Nemo-K GNSS NEO 6M-V2 v3 (C) Sivuduuni Global Oy 2025"
- board text added: "VCC"
- board text removed: "Nemo-K GNSS NEO 6M-V2 v2 (C) Sivuduuni Global Oy 2025"
