File: sensor-gnss-neo6mv2/sensor-gnss-neo6mv2.kicad_sch (KiCad schematic)
At the start: 7 parts, among them J1 PWR, J2 ESP-01S, J3 NEO6M, U1 LMZM23601V3SILR

Commit message: First prototype sent to production
Parts:
- D1: LCSC (none) -> C5174649
- J3: LCSC C5160786 -> C42379197
Connections:
- net at J3.2 (RX): no longer J2.2 (TX)
- net Data: now reaches J2.7 (RX), J3.3 (TX)
- net PWR VCC: now reaches D1.2 (A), J1.1 (VCC)
Other:
- moved on the sheet: J2
Changed lines of the file:
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@@
 	)
 	(junction
-		(at 158.75 146.05)
+		(at 191.77 115.57)
 		(diameter 0)
 		(color 0 0 0 0)
@@
 	(wire
 		(pts
-			(xy 130.81 151.13) (xy 138.43 151.13)
-		)
-		(stroke
-			(width 0)
-			(type default)
-		)
-	)
-	(wire
-		(pts
 			(xy 135.89 87.63) (xy 123.19 87.63)
 		)
@@
 	(wire
 		(pts
-			(xy 152.4 143.51) (xy 152.4 133.35)
-		)
-		(stroke
-			(width 0)
-			(type default)
-		)
-	)
-	(wire
-		(pts
 			(xy 138.43 120.65) (xy 135.89 120.65)
 		)
@@
 	(wire
 		(pts
-			(xy 148.59 143.51) (xy 152.4 143.51)
-		)
-		(stroke
-			(width 0)
-			(type default)
-		)
-	)
-	(wire
-		(pts
 			(xy 180.34 86.36) (xy 180.34 96.52)
 		)
@@
 	(wire
 		(pts
-			(xy 158.75 140.97) (xy 158.75 146.05)
+			(xy 191.77 110.49) (xy 191.77 115.57)
 		)
 		(stroke
@@
 	(wire
 		(pts
-			(xy 148.59 120.65) (xy 148.59 130.81)
-		)
-		(stroke
-			(width 0)
-			(type default)
-		)
-	)
-	(wire
-		(pts
-			(xy 134.62 143.51) (xy 138.43 143.51)
+			(xy 167.64 113.03) (xy 171.45 113.03)
 		)
 		(stroke
@@
 	(wire
 		(pts
-			(xy 133.35 133.35) (xy 133.35 118.11)
-		)
-		(stroke
-			(width 0)
-			(type default)
-		)
-	)
-	(wire
-		(pts
-			(xy 130.81 130.81) (xy 148.59 130.81)
-		)
-		(stroke
-			(width 0)
-			(type default)
-		)
-	)
-	(wire
-		(pts
-			(xy 148.59 146.05) (xy 158.75 146.05)
+			(xy 181.61 115.57) (xy 191.77 115.57)
 		)
 		(stroke
@@
 	(wire
 		(pts
-			(xy 158.75 146.05) (xy 158.75 151.13)
-		)
-		(stroke
-			(width 0)
-			(type default)
-		)
-	)
-	(wire
-		(pts
-			(xy 152.4 133.35) (xy 133.35 133.35)
+			(xy 191.77 115.57) (xy 191.77 120.65)
+		)
+		(stroke
+			(width 0)
+			(type default)
+		)
+	)
+	(wire
+		(pts
+			(xy 148.59 120.65) (xy 171.45 120.65)
 		)
 		(stroke
@@
 	(wire
 		(pts
-			(xy 130.81 130.81) (xy 130.81 151.13)
-		)
-		(stroke
-			(width 0)
-			(type default)
-		)
-	)
-	(wire
-		(pts
 			(xy 193.04 77.47) (xy 193.04 76.2)
 		)
@@
 	(wire
 		(pts
-			(xy 134.62 156.21) (xy 134.62 143.51)
+			(xy 167.64 125.73) (xy 167.64 113.03)
 		)
 		(stroke
@@
 	(wire
 		(pts
-			(xy 158.75 151.13) (xy 148.59 151.13)
+			(xy 191.77 120.65) (xy 181.61 120.65)
 		)
 		(stroke
@@
 	(wire
 		(pts
-			(xy 133.35 118.11) (xy 138.43 118.11)
-		)
-		(stroke
-			(width 0)
-			(type default)
-		)
-	)
-	(wire
-		(pts
 			(xy 151.13 118.11) (xy 151.13 115.57)
 		)
@@
 			(width 0)
 			(type default)
+		)
+	)
+	(label "Data"
+		(at 157.48 120.65 0)
+		(effects
+			(font
+				(size 1.27 1.27)
+			)
+			(justify left bottom)
+		)
+	)
+	(label "PWR VCC"
+		(at 93.98 77.47 0)
+		(effects
+			(font
+				(size 1.27 1.27)
+			)
+			(justify left bottom)
 		)
 	)
@@
 			)
 		)
-		(property "LCSC" "C5160786"
+		(property "LCSC" "C42379197"
 			(at 143.51 119.38 0)
 			(effects
@@
 	(symbol
 		(lib_id "C3975149:PM254-2-04-S-8.5")
-		(at 143.51 147.32 0)
+		(at 176.53 116.84 0)
 		(mirror y)
 		(unit 1)
@@
 		(fields_autoplaced yes)
 		(property "Reference" "J2"
-			(at 143.51 135.89 0)
+			(at 176.53 105.41 0)
 			(effects
 				(font
@@
 		)
 		(property "Value" "ESP-01S"
-			(at 143.51 138.43 0)
+			(at 176.53 107.95 0)
 			(effects
 				(font
@@
 		)
 		(property "Footprint" "C3975149:HDR-SMD_8P-P2.54-V-F-R2-C4-S7.1"
-			(at 143.51 147.32 0)
+			(at 176.53 116.84 0)
 			(effects
 				(font
@@
 		)
 		(property "Datasheet" "https://atta.szlcsc.com/upload/public/pdf/source/20230609/7C6F8D8E301C6BBC8F19D55951C36597.pdf"
-			(at 143.51 147.32 0)
+			(at 176.53 116.84 0)
 			(effects
 				(font
@@
 		)
 		(property "Description" "Holes Structure:2x4P Pitch:2.54mm Row Spacing:2.54mm Circular Hole / Square Hole:方孔 Mounting Type:Brick nogging Number of Rows:双排 Number of Holes:8P Current Rating (Max):3A Holes Direction:Top Insulation Height:8.5mm Contact Material:Copper Alloy Operatin"
-			(at 143.51 147.32 0)
+			(at 176.53 116.84 0)
 			(effects
 				(font
@@
 		)
 		(property "LCSC" "C3975149"
-			(at 143.51 147.32 0)
+			(at 176.53 116.84 0)
 			(effects
 				(font
@@
 		)
 		(property "Mfg Part" "PM254-2-04-S-8.5"
-			(at 143.51 147.32 0)
+			(at 176.53 116.84 0)
 			(effects
 				(font
@@
 		)
 		(property "Manufacturer Part" "PM254-2-04-S-8.5"
-			(at 143.51 147.32 0)
+			(at 176.53 116.84 0)
 			(effects
 				(font
@@
 		)
 		(property "Manufacturer" "HCTL(华灿天禄)"
-			(at 143.51 147.32 0)
+			(at 176.53 116.84 0)
 			(effects
 				(font
@@
 		)
 		(property "Supplier Part" "C3975149"
-			(at 143.51 147.32 0)
+			(at 176.53 116.84 0)
 			(effects
 				(font
@@
 		)
 		(property "Supplier" "LCSC"
-			(at 143.51 147.32 0)
+			(at 176.53 116.84 0)
 			(effects
 				(font
@@
 		)
 		(property "LCSC Part Name" "2x4P 间距:2.54mm 立贴"
-			(at 143.51 147.32 0)
+			(at 176.53 116.84 0)
 			(effects
 				(font
@@
 		)
 		(property "LCSC Part Name" "S7116-300A"
+			(at 102.87 77.47 0)
+			(effects
+				(font
+					(size 1.27 1.27)
+				)
+				(hide yes)
+			)
+		)
+		(property "LCSC" "C5174649"
 			(at 102.87 77.47 0)
 			(effects
@@
 	(symbol
 		(lib_id "power:+3V3")
-		(at 158.75 140.97 0)
+		(at 191.77 110.49 0)
 		(unit 1)
 		(exclude_from_sim no)
@@
 		(fields_autoplaced yes)
 		(property "Reference" "#PWR0107"
-			(at 158.75 144.78 0)
+			(at 191.77 114.3 0)
 			(effects
 				(font
@@
 		)
 		(property "Value" "+3V3"
-			(at 158.75 135.89 0)
+			(at 191.77 105.41 0)
 			(effects
 				(font
@@
 		)
 		(property "Footprint" ""
-			(at 158.75 140.97 0)
+			(at 191.77 110.49 0)
 			(effects
 				(font
@@
 		)
 		(property "Datasheet" ""
-			(at 158.75 140.97 0)
+			(at 191.77 110.49 0)
 			(effects
 				(font
@@
 		)
 		(property "Description" ""
-			(at 158.75 140.97 0)
+			(at 191.77 110.49 0)
 			(effects
 				(font
@@
 	(symbol
 		(lib_id "power:Earth")
-		(at 134.62 156.21 0)
+		(at 167.64 125.73 0)
 		(unit 1)
 		(exclude_from_sim no)
@@
 		(fields_autoplaced yes)
 		(property "Reference" "#PWR0104"
-			(at 134.62 162.56 0)
+			(at 167.64 132.08 0)
 			(effects
 				(font
@@
 		)
 		(property "Value" "Earth"
-			(at 134.62 160.02 0)
+			(at 167.64 129.54 0)
 			(effects
 				(font
@@
 		)
 		(property "Footprint" ""
-			(at 134.62 156.21 0)
+			(at 167.64 125.73 0)
 			(effects
 				(font
@@
 		)
 		(property "Datasheet" "~"
-			(at 134.62 156.21 0)
+			(at 167.64 125.73 0)
 			(effects
 				(font
@@
 		)
 		(property "Description" ""
-			(at 134.62 156.21 0)
-			(effects
-				(font
+			(at 167.64 125.73 0)
+			(effects
+				(font

Commit message: v3, revised based on first proto version
Parts:
- J1: footprint TerminalBlock_MetzConnect:TerminalBlock_MetzConnect_Type086_RT03402HBLC_1x02_P3.81mm_Horizontal -> C5349550:CONN-TH_MX127S-3.81-02P-GN01-CU-Y-A; symbol Connector:Screw_Terminal_01x02 -> C5349550:MX127S-3.81-02P-GN01-CU-Y-A; LCSC Part Name (none) -> 1x2P 3.81mm 直插 排数:1 每排P数:2; Manufacturer (none) -> MAX(迈旭); Manufacturer Part (none) -> MX127S-3.81-02P-GN01-Cu-Y-A; Supplier (none) -> LCSC; Supplier Part (none) -> C5349550
Changed lines of the file:
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@@
 	(title_block
 		(title "Nemo-K NEO6MV2 sensor")
-		(date "2025-10-08")
-		(rev "v2")
+		(date "2025-11-15")
+		(rev "v3")
 		(company "Sivuduuni Global Oy")
 	)
@@
 	)
 	(symbol
-		(lib_id "Connector:Screw_Terminal_01x02")
-		(at 88.9 77.47 0)
+		(lib_id "C5349550:MX127S-3.81-02P-GN01-CU-Y-A")
+		(at 88.9 78.74 0)
 		(mirror y)
 		(unit 1)
@@
 		(fields_autoplaced yes)
 		(property "Reference" "J1"
-			(at 88.9 71.12 0)
+			(at 88.9 69.85 0)
 			(effects
 				(font
@@
 		)
 		(property "Value" "PWR"
-			(at 88.9 73.66 0)
-			(effects
-				(font
-					(size 1.27 1.27)
-				)
-			)
-		)
-		(property "Footprint" "TerminalBlock_MetzConnect:TerminalBlock_MetzConnect_Type086_RT03402HBLC_1x02_P3.81mm_Horizontal"
-			(at 88.9 77.47 0)
-			(effects
-				(font
-					(size 1.27 1.27)
-				)
-				(hide yes)
-			)
-		)
-		(property "Datasheet" "~"
-			(at 88.9 77.47 0)
-			(effects
-				(font
-					(size 1.27 1.27)
-				)
-				(hide yes)
-			)
-		)
-		(property "Description" "Generic screw terminal, single row, 01x02, script generated (kicad-library-utils/schlib/autogen/connector/)"
-			(at 88.9 77.47 0)
+			(at 88.9 72.39 0)
+			(effects
+				(font
+					(size 1.27 1.27)
+				)
+			)
+		)
+		(property "Footprint" "C5349550:CONN-TH_MX127S-3.81-02P-GN01-CU-Y-A"
+			(at 88.9 78.74 0)
+			(effects
+				(font
+					(size 1.27 1.27)
+				)
+				(hide yes)
+			)
+		)
+		(property "Datasheet" "https://atta.szlcsc.com/upload/public/pdf/source/20230914/FF202AD9F8A47F92BC9493963328A9C4.pdf"
+			(at 88.9 78.74 0)
+			(effects
+				(font
+					(size 1.27 1.27)
+				)
+				(hide yes)
+			)
+		)
+		(property "Description" "Structure:1x2P Pitch:3.81mm Color:Green Mounting Style:Direct Insert Number of Pins:2P Number of Rows:1 Number of PINs Per Row:2 Screw Specification:M2 Current Rating (Max):10A Voltage Rating (Max):300V Wire Gauge - AWG:16~26 Wire Gauge - AWG:16~26 Operat"
+			(at 88.9 78.74 0)
 			(effects
 				(font
@@
 		)
 		(property "LCSC" "C5349550"
-			(at 88.9 77.47 0)
+			(at 88.9 78.74 0)
 			(effects
 				(font
@@
 		)
 		(property "MPN" "OSTOQ053251"
-			(at 88.9 77.47 0)
-			(effects
-				(font
+			(at 88.9 78.74 0)
+			(effects
+				(font
+					(size 1.27 1.27)
+				)
+				(hide yes)
+			)
+		)
+		(property "Manufacturer Part" "MX127S-3.81-02P-GN01-Cu-Y-A"
+			(at 88.9 78.74 0)
+			(effects
+				(font
+					(size 1.27 1.27)
+				)
+				(hide yes)
+			)
+		)
+		(property "Manufacturer" "MAX(迈旭)"
+			(at 88.9 78.74 0)
+			(effects
+				(font
+					(size 1.27 1.27)
+				)
+				(hide yes)
+			)
+		)
+		(property "Supplier Part" "C5349550"
+			(at 88.9 78.74 0)
+			(effects
+				(font
+					(size 1.27 1.27)
+				)
+				(hide yes)
+			)
+		)
+		(property "Supplier" "LCSC"
+			(at 88.9 78.74 0)
+			(effects
+				(font
+					(size 1.27 1.27)
+				)
+				(hide yes)
+			)
+		)
+		(property "LCSC Part Name" "1x2P 3.81mm 直插 排数:1 每排P数:2"
+			(at 88.9 78.74 0)
+			(effects
+				(font
